Commit message: Added final docking logic based on aruco marker yaw angles

File: turtlebot3_gazebo/urdf/turtlebot3_waffle.urdf (robot description, URDF)
Before this commit: robot turtlebot3_waffle, 13 links, 12 joints
Joints:
- joint camera_joint: origin xyz=0.064 -0.065 0.094 rpy=0 0 0 -> xyz=0.064 0.0 0.094 rpy=0 0 0
- joint camera_rgb_joint: origin xyz=0.005 0.018 0.013 rpy=0 0 0 -> xyz=-0.001 0.00 0.00 rpy=0 0 0

Commit message: Aruco size change, camera joint position correcetd

File: turtlebot3_gazebo/urdf/turtlebot3_waffle.urdf (robot description, URDF)
Before this commit: robot turtlebot3_waffle, 13 links, 12 joints
Joints:
- joint camera_rgb_joint: origin xyz=-0.001 0.00 0.00 rpy=0 0 0 -> xyz=-0.00 0.00 0.00 rpy=0 0 0

Commit message: Added depth camera with point cloud

File: turtlebot3_gazebo/urdf/turtlebot3_waffle.urdf (robot description, URDF)
Before this commit: robot turtlebot3_waffle, 13 links, 12 joints
Joints:
- joint camera_depth_joint: origin xyz=0.005 0.028 0.013 rpy=0 0 0 -> xyz=0.0 0.0 0.0 rpy=1.5708 -3.14 1.5708
